File: sensors/moist/moist/moist.kicad_sch (KiCad schematic)
At the start: 3 parts

Commit message: moist sensor schematic
Parts:
- added C1, C4: 100n, symbol Device:C
- added C2: 1u, symbol Device:C
- added J2: Conn_01x02, symbol Connector_Generic:Conn_01x02
- added R1: 1k, symbol Device:R
- added R?: R, symbol Device:R
- added U1: TL431D, Package_SO:SOIC-8_3.9x4.9mm_P1.27mm, symbol Reference_Voltage:TL431D
- added U?: LM358, symbol Amplifier_Operational:LM358
- gave numbers to parts that had none: 3
Connections:
- net at U4.1: now also U2.2 (IN+), U4.2 (-)
- net at U4.3 (+): now also J2.1 (Pin_1), R?.2
- net GND: now reaches J1.1 (Pin_1)
- net GND: now also U2.3 (IN-), U2.4 (Vss), C1.2, C2.2, C4.2, J2.2 (Pin_2), U1.2 (A), U1.3 (A), U1.6 (A), U1.7 (A), U?.4 (V-)
- net at J1.2 (Pin_2): now also U2.7 (CLK)
- net at J1.3 (Pin_3): now also U2.6 (Dout)
- net at J1.4 (Pin_4): now also U2.5 (~{CS}/SHDN)
- net +5P: now reaches J1.5 (Pin_5)
- net +5P: now also U2.8 (Vdd), C2.1, C4.1, R1.1, R?.1, U?.8 (V+)
- net at U2.1 (Vref): now also C1.1, R1.2, U1.1 (K), U1.8 (REF)
Other:
- moved on the sheet: J1, U4A
